File: ecad/riskybird.kicad_sch (KiCad schematic)
At the start: 80 parts, among them J1 USB_B_Micro, J2 Conn_01x02, J3 Conn_01x02, J4 Conn_01x02, J5 Conn_01x02, J6 Conn_01x02, J7 Conn_01x10, J8 Conn_01x10, Q1 SI2302, Q2 SI2302, Q3 SI2302, Q4 SI2302, Q5 DNBT8105-7, Q6 DNBT8105-7, Q7 Q_NMOS_GSD, SW1 SW_SPST, SW2 SW_SPST, SW3 SW_SPST, U1 MCP73831-2-OT, U10 74LVC2G08, U3 TPS2113A, U4 LP2985-3.0, U6 ESP32-C3-WROOM-02, U7 BMI088, U8 FT231XS

Commit message: RiskyBird 0.1
Parts:
- removed C14, C15, C7: 0.1u, Capacitor_SMD:C_0603_1608Metric_Pad1.08x0.95mm_HandSolder, symbol Device:C
- removed C16: 10u, Capacitor_SMD:C_0603_1608Metric_Pad1.08x0.95mm_HandSolder, symbol Device:C
- removed Q5, Q6: DNBT8105-7, Package_TO_SOT_SMD:SOT-23, symbol Device:Q_NPN_BEC
- removed R23: 10k, Resistor_SMD:R_0603_1608Metric_Pad0.98x0.95mm_HandSolder, symbol Device:R
- removed U10: 74LVC2G08, Package_SO:VSSOP-8_3.0x3.0mm_P0.65mm, symbol 74xGxx:74LVC2G08
- removed U6: ESP32-C3-WROOM-02, Espressif:ESP32-C3-WROOM-02, symbol Espressif:ESP32-C3-WROOM-02
- added C5: 10u, Capacitor_SMD:C_0402_1005Metric, symbol Device:C
- added C6, C8: 0.1u, Capacitor_SMD:C_0402_1005Metric, symbol Device:C
- added Q8: BC847BDW1, Package_TO_SOT_SMD:SOT-363_SC-70-6, symbol Transistor_BJT:BC847BDW1
- added R26: 10k, Resistor_SMD:R_0402_1005Metric, symbol Device:R
- added U5: ESP32-C6-MINI-1/U, Espressif:ESP32-C6-MINI-1, symbol Espressif:ESP32-C6-MINI-1/U
- C1, C10, C11, C12, C13, C17, C18, C19, C2, C20, C21, C3, C4: footprint Capacitor_SMD:C_0603_1608Metric_Pad1.08x0.95mm_HandSolder -> Capacitor_SMD:C_0402_1005Metric
- L1: footprint Inductor_SMD:L_0805_2012Metric_Pad1.15x1.40mm_HandSolder -> Inductor_SMD:L_0402_1005Metric
- R1, R10, R11, R12, R13, R14, R15, R16, R17, R18, R19, R2, R20, R21, R22, R24, R25, R3, R4, R5, R6, R7, R8, R9: footprint Resistor_SMD:R_0603_1608Metric_Pad0.98x0.95mm_HandSolder -> Resistor_SMD:R_0402_1005Metric
- U2: footprint riskybird:BMP390_Handsolder -> riskybird:BMP390
- U7: footprint riskybird:BMI088_Handsolder -> riskybird:BMI088
Connections:
- net CHIP_EN: now also C8.1, Q8.3 (C2), U5.8 (EN/CHIP_PU)
- net DTR: now also Q8.1 (E1)
- net GND: now also R4.2
- net GNDD: now also C5.2, C6.2, C8.2, U5.1 (GND), U5.11 (GND), U5.14 (GND), U5.2 (GND), U5.36 (GND), U5.37 (GND), U5.38 (GND), U5.39 (GND), U5.40 (GND), U5.41 (GND), U5.42 (GND), U5.43 (GND), U5.44 (GND), U5.45 (GND), U5.46 (GND), U5.47 (GND), U5.48 (GND), U5.49 (GND), U5.50 (GND), U5.51 (GND), U5.52 (GND), U5.53 (GND); no longer R4.2
- net GPIO9: now also Q8.6 (C1), U5.23 (GPIO9)
- net MOTOR1: now also U5.26 (GPIO20)
- net MOTOR2: now also U5.27 (GPIO21)
- net MOTOR3: now also U5.28 (GPIO22)
- net MOTOR4: now also U5.29 (GPIO23)
- net OW: now also U5.13 (GPIO1/ADC1_CH1/XTAL_32K_N)
- net RGB_CTRL: now also R26.2, U5.22 (GPIO8)
- net RTS: now also Q8.4 (E2)
- net SCL: now also R8.2, U5.19 (GPIO14); no longer R9.2
- net SDA: now also R9.2, U5.20 (GPIO15); no longer R8.2
- net U0RXD: now also U5.30 (U0RXD/GPIO17)
- net U0TXD: now also U5.31 (U0TXD/GPIO16)
- net U1RXD: now also U5.17 (GPIO12/USB_D-)
- net U1TXD: now also U5.18 (GPIO13/USB_D+)
- net VCOM: no longer Q7.1 (G)
- net VDD: now also Q7.1 (G), C5.1, C6.1, R26.1, U5.3 (3V3)
- net VSENSE: now also U5.12 (GPIO0/ADC1_CH0/XTAL_32K_P)
- net SCK: now reaches J8.3 (Pin_3)
- net SCK: now also U5.15 (MTCK/GPIO6/ADC1_CH6)
- net MISO: now reaches J8.4 (Pin_4)
- net MISO: now also U5.24 (GPIO18)
- net MOSI: now reaches J8.5 (Pin_5)
- net MOSI: now also U5.16 (MTDO/GPIO7)
- net IO5: now reaches J8.6 (Pin_6)
- net IO5: now also U5.25 (GPIO19)
- net at R20.2: now also Q8.5 (B2)
- net IO1: now reaches J7.6 (Pin_6)
- net IO1: now also U5.10 (MTDI/GPIO5/ADC1_CH5)
- net IO2: now reaches J7.7 (Pin_7)
- net IO2: now also U5.9 (MTMS/GPIO4/ADC1_CH4)
- net IO3: now reaches J7.8 (Pin_8)
- net IO3: now also U5.6 (GPIO3/ADC1_CH3)
- net IO4: now reaches J7.9 (Pin_9)
- net IO4: now also U5.5 (GPIO2/ADC1_CH2)
- net at R21.2: now also Q8.2 (B1)
- net INT_ACC: no longer names the net of U7.16 (INT1)
- net INT_BARO: no longer names the net of U2.7 (INT)
- net INT_GYR: no longer names the net of U7.1 (INT2)
- net INT_GYR: no longer U7.12 (INT3)
- no-connect marks 23 -> 19
